File: kicad/kit/an043_ref/kit_an043_ref.kicad_sch (KiCad schematic)
At the start: 5 parts, among them J1 SMA edge launch

Commit message: Kit launches through U.FL and a pigtail, not an SMA on the board edge
Embever's own antenna kit feeds its boards through a U.FL and a pigtail
to a bulkhead SMA. That is the better arrangement for a measurement kit
and the kit now does it.

The connector is the smaller half of the reason. The real one is that on
a 45 x 60 mm plane at 868 MHz - lambda 345 mm - the plane and whatever
cable leaves it are one conductor as far as common-mode current goes, so
the braid is part of the antenna and the S11 null moves when the cable
moves. Nothing about the connector fixes that. What U.FL does is let you
fix it: the bulkhead SMA stays on the jig instead of leaving a connector
shell and its ground tabs as copper beside a plane that is half the
antenna, and the pigtail is somewhere to put a ferrite or a sleeve balun,
which is the only real cure. The checklist and the measurement procedure
now both start with choking the cable and proving it by moving it.

The land pattern is Hirose's own for the U.FL-R-SMT-1(10) - signal pad
1.05 x 1.00, ground pads 2.20 x 1.05 - taken from KiCad's
Connector_Coaxial library, which cites Hirose's page for the part. It is
regenerated from those dimensions rather than copied, so the provenance
sits next to the geometry; KiCad's libraries are CC-BY-SA 4.0 with a
design exception and this is the attribution.

A 1.05 mm pad will not take a 2.95 mm line, the same trap the through-
hole SMA sprang with its ground posts. The line tapers 2.95 -> 1.0 mm
over 2.5 mm and runs 1.5 mm into the pad, and the pour keep-away now
stops above the connector so the pour closes around J1's ground pads.
That turns the neck into a grounded coplanar line instead of a
microstrip: line_impedance.py puts 1.0 mm with a 0.2 mm gap at 53.9 ohm
against 84.5 ohm bare, so the neck is near 50 ohm by construction rather
than a lump for the network to absorb.

The launch needed its own rules, because the general ones do not cover
it: a track and the pad it runs to are the same net, s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
Parts:
- J1: value SMA edge launch -> U.FL receptacle; footprint SWRA117D_RF:SMA_EdgeMount_Generic -> SWRA117D_RF:U_FL_Hirose_U_FL_R_SMT_1_Vertical
Other:
- note added: "Antenna evaluation kit, board an043_ref. Antenna: AN043 / SWRA117D, 2450 MHz, an exact copy of the note's own dimension table, checked by its verify_against_* script. Ground plane: 40 x 28 mm, this repo's own choice - the note publishes no plane size. Matching: Z1=DNP Z2=0R Z3=DNP SWRA117D publishes no matching values and no ground plane size. The plane here is this repo's own 40 x 23.75 mm, not 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"
- note removed: "Antenna evaluation kit, board an043_ref. Antenna: AN043 / SWRA117D, 2450 MHz, an exact copy of the note's own dimension table, checked by its verify_against_* script. Ground plane: 40 x 23.75 mm, this repo's own choice - the note publishes no plane size. Matching: Z1=DNP Z2=0R Z3=DNP SWRA117D publishes no matching values and no ground plane size. The plane here is this repo's own 40 x 23.75 mm, n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"
- title: TI AN043 / SWRA117D on a 40 x 23.75 mm reference plane -> TI AN043 / SWRA117D on a 40 x 28 mm reference plane
Changed lines of the file:
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@@
 	(paper "A4")
 	(title_block
-		(title "TI AN043 / SWRA117D on a 40 x 23.75 mm reference plane")
+		(title "TI AN043 / SWRA117D on a 40 x 28 mm reference plane")
 		(date "2026-09-12")
 		(rev "A")
@@
 		(effects (font (size 1.27 1.27)) (justify left bottom))
 	)
-	(text "Antenna evaluation kit, board an043_ref.\n\nAntenna: AN043 / SWRA117D, 2450 MHz, an exact copy of the note's\nown dimension table, checked by its verify_against_* script.\n\nGround plane: 40 x 23.75 mm, this repo's own choice - the note publishes no plane size.\n\nMatching: Z1=DNP  Z2=0R  Z3=DNP\nSWRA117D publishes no matching values and no ground plane size. The plane here is this repo's own 40 x 23.75 mm, not TI's - the note only says plane size affects performance.\n\n2.95 mm wide 50 ohm microstrip on 1.6 mm FR4 (er 4.5),\nthe same on all six boards so the launch is not a variable.\n\nBefore simulating or running DRC: fill the zones (B in the PCB\neditor). KiCad stores them unfilled and a plane is half the antenna."
+	(text "Antenna evaluation kit, board an043_ref.\n\nAntenna: AN043 / SWRA117D, 2450 MHz, an exact copy of the note's\nown dimension table, checked by its verify_against_* script.\n\nGround plane: 40 x 28 mm, this repo's own choice - the note publishes no plane size.\n\nMatching: Z1=DNP  Z2=0R  Z3=DNP\nSWRA117D publishes no matching values and no ground plane size. The plane here is this repo's own 40 x 23.75 mm, not TI's - the note only says plane size affects performance.\n\n2.95 mm wide 50 ohm microstrip on 1.6 mm FR4 (er 4.5),\nthe same on all six boards so the launch is not a variable.\n\nBefore simulating or running DRC: fill the zones (B in the PCB\neditor). KiCad stores them unfilled and a plane is half the antenna."
 		(exclude_from_sim no)
 		(at 76.2 112 0)
@@
 		(dnp no)
 		(property "Reference" "J1" (at 63.5 81.28 0) (effects (font (size 1.27 1.27)) (justify left)))
-		(property "Value" "SMA edge launch"
+		(property "Value" "U.FL receptacle"
 			(at 63.5 83.82 0)
 			(effects (font (size 1.27 1.27)) (justify left))
 		)
-		(property "Footprint" "SWRA117D_RF:SMA_EdgeMount_Generic"
+		(property "Footprint" "SWRA117D_RF:U_FL_Hirose_U_FL_R_SMT_1_Vertical"
 			(at 63.5 88.9 0)
 			(effects (font (size 1.27 1.27)) (hide yes))
 		)
 		(property "Datasheet" "~" (at 63.5 88.9 0) (effects (font (size 1.27 1.27)) (hide yes)))
-		(property "Description" "Coaxial connector, 50 ohm test port. The same part on all six boards, so the launch is not a variable"
+		(property "Description" "Hirose U.FL-R-SMT-1(10), fed by a pigtail to a bulkhead SMA on the jig. The same part on all six boards, so the launch is not a variable. Put a ferrite or a sleeve balun on the pigtail: on a plane this size the cable braid is part of the antenna until you choke it"
 			(at 63.5 88.9 0)
 			(effects (font (size 1.27 1.27)) (hide yes))
